File: pcb/usb.kicad_sch (KiCad schematic)
At the start: 31 parts, among them J17 USB_B_Mini, Q22 PMOS, Q23 PMOS, Q25 NMOS, Q27 PMOS, U15 FT230XQ, U19 PUSBM5V5X4-TL_115

Commit message: Update PCB to new KiCAD version, Fix repair notes about U23, add part number for L2, and update IMU firmware information
Parts:
- L2: value 0603USB-251 -> ACM-0603-900-T
Other:
- note removed: "L2 is an educated guess"
